File: Hardware/UNO_Q_Breakout/UNO_Q_Breakout.kicad_sch (KiCad schematic)
At the start: 3 parts, among them J1 Conn_02x30_Odd_Even, J2 LAMP1

Commit message: Update floorplan
Connections:
- net MCU_SDMMC1_CMD: now reaches J1.1 (Pin_1)
- net MCU_PSSI_D4: now reaches J1.10 (Pin_10)
- net MCU_PSSI_D5: now reaches J1.12 (Pin_12)
- net MCU_PSSI_D6: now reaches J1.14 (Pin_14)
- net MCU_PSSI_D7: now reaches J1.16 (Pin_16)
- net MCU_PSSI_PDCK: now reaches J1.18 (Pin_18)
- net MCU_PSSI_D0: now reaches J1.2 (Pin_2)
- net MCU_PSSI_RDY: now reaches J1.20 (Pin_20)
- net MCU_PSSI_DE: now reaches J1.22 (Pin_22)
- net MCU_MCO: now reaches J1.24 (Pin_24)
- net MCU_CRS_SYNC: now reaches J1.26 (Pin_26)
- net MCU_PSSI_D1: now reaches J1.4 (Pin_4)
- net MCU_PSSI_D2: now reaches J1.6 (Pin_6)
- net MCU_PSSI_D3: now reaches J1.8 (Pin_8)
- no-connect marks 51 -> 37
