File: Hardware/UNO_Q_Breakout/UNO_Q_Breakout.kicad_pcb (KiCad board)
At the start: 2 copper layers, 11 x 56 mm, 3 parts, among them J1 Conn_02x30_Odd_Even, J2 LAMP1

Commit message: Update floorplan
Parts:
- moved J2 22.4 mm to (150.0, 60.5), turned to 90 degrees
- moved JP1 20.3 mm to (151.7, 60.8)
Connections:
- J1 pad 1: unconnected-(J1-Pin_1-Pad1) -> /MCU_SDMMC1_CMD
- J1 pad 10: unconnected-(J1-Pin_10-Pad10) -> /MCU_PSSI_D4
- J1 pad 12: unconnected-(J1-Pin_12-Pad12) -> /MCU_PSSI_D5
- J1 pad 14: unconnected-(J1-Pin_14-Pad14) -> /MCU_PSSI_D6
- J1 pad 16: unconnected-(J1-Pin_16-Pad16) -> /MCU_PSSI_D7
- J1 pad 18: unconnected-(J1-Pin_18-Pad18) -> /MCU_PSSI_PDCK
- J1 pad 2: unconnected-(J1-Pin_2-Pad2) -> /MCU_PSSI_D0
- J1 pad 20: unconnected-(J1-Pin_20-Pad20) -> /MCU_PSSI_RDY
- J1 pad 22: unconnected-(J1-Pin_22-Pad22) -> /MCU_PSSI_DE
- J1 pad 24: unconnected-(J1-Pin_24-Pad24) -> /MCU_MCO
- J1 pad 26: unconnected-(J1-Pin_26-Pad26) -> /MCU_CRS_SYNC
- J1 pad 4: unconnected-(J1-Pin_4-Pad4) -> /MCU_PSSI_D1
- J1 pad 6: unconnected-(J1-Pin_6-Pad6) -> /MCU_PSSI_D2
- J1 pad 8: unconnected-(J1-Pin_8-Pad8) -> /MCU_PSSI_D3
Routing:
- net +1V8: track 64.9 -> 0.00 mm, vias 2 -> 0
- net /MIC_M: track 39.8 -> 0.00 mm, vias 1 -> 0
- net /MIC_P: track 36.5 -> 0.00 mm, vias 1 -> 0
- net /MIC_BIAS: track 28.6 -> 0.00 mm
- net /MIC_BIAS_O: track 10.5 -> 0.00 mm, vias 1 -> 0
- net GND: vias 6 -> 0
- removed copper zone on B.Cu, net GND
- removed copper zone on F.Cu, net GND
Other:
- board size 11 x 56 mm -> 23 x 41 mm
- board text added: "1"

Commit message: Update Hardware
Parts:
- moved JP1 20.0 mm to (131.8, 60.5)
- moved J2 18.1 mm to (131.9, 60.5), turned to -90 degrees
Routing:
- net +1V8: track 0.00 -> 41.0 mm, vias 0 -> 1
- net /MIC_M: track 0.00 -> 18.5 mm, vias 0 -> 1
- net /MIC_BIAS: track 0.00 -> 15.3 mm, vias 0 -> 1
- net /MIC_P: track 0.00 -> 15.0 mm, vias 0 -> 1
- net /MIC_BIAS_O: track 0.00 -> 9.15 mm, vias 0 -> 1
- net GND: track 0.00 -> 4.22 mm, vias 0 -> 2
- added copper zone on B.Cu, net GND
- added copper zone on F.Cu, net GND
Other:
- board size 23 x 41 mm -> 15.5 x 41 mm
- board text added: "1.8v"
