File: Hardware/UNO_Q_Breakout/UNO_Q_Breakout.kicad_pcb (KiCad board)
At the start: 2 copper layers, 15.5 x 41 mm, 3 parts, among them J1 Conn_02x30_Odd_Even, J2 LAMP1

Commit message: Update hardware projects for Gerber generation
- Configure Gerber output directories for Microphone, QWIIC LEDs, and UNO Q Breakout projects.
- Update .gitignore to exclude Gerber and drill files.
- Refine PCB layouts and update versioning labels for production readiness.
Other:
- board text added: "UNO_Q_Breakout v1.0"
- board text removed: "GND"
- board text removed: "MIC +"
- board text removed: "MIC -"
- board text removed: "MIC BIAS"
